Commit message: Updated models

File: src/r1_2020/urdf/r1_2020.urdf (robot description, URDF)
Before this commit: robot r1_2020, 3 links, 2 joints
Joints:
- joint left_wheel_joint: origin xyz=0 0 0 rpy=0 0 0 -> xyz=0 0.16056 0.079717 rpy=0 0 0
- joint right_wheel_joint: origin xyz=0 0 0 rpy=0 0 0 -> xyz=0 -0.16644 0.079717 rpy=0 0 0

File: src/r2_2020/urdf/r2_2020.urdf (robot description, URDF)
Before this commit: robot r2_2020, 4 links, 3 joints
Links:
- link base_link: mass 9.9402 -> 9.9293
Joints:
- joint left_wheel_joint: origin xyz=0 0 0 rpy=0 0 0 -> xyz=-0.11755 0.1805 0.0655 rpy=0 0 0
- joint right_wheel_joint: origin xyz=0 0 0 rpy=0 0 0 -> xyz=-0.11755 -0.1805 0.0655 rpy=0 0 0
- joint weapon_joint: origin xyz=0 0 0 rpy=0 0 0 -> xyz=0.2077 0.00068787 0.179 rpy=0 0 0

File: src/r3_2020/urdf/r3_2020.urdf (robot description, URDF)
Before this commit: robot r3_2020, 5 links, 4 joints
Joints:
- joint blade_left_joint: origin xyz=0 0 0 rpy=0 0 0 -> xyz=0.3015 0.1503 0.13348 rpy=0 0 0
- joint blade_right_joint: origin xyz=0 0 0 rpy=0 0 0 -> xyz=0.3015 -0.1503 0.13348 rpy=0 0 0
- joint wheel_left_link: origin xyz=0 0 0 rpy=0 0 0 -> xyz=0.0014732 0.17376 0.051477 rpy=0 0 0
- joint wheel_right_joint: origin xyz=0 0 0 rpy=0 0 0 -> xyz=-0.0014732 -0.17376 0.051477 rpy=0 0 0

File: src/r4_2020/urdf/r4_2020.urdf (robot description, URDF)
Before this commit: robot r4_2020, 3 links, 2 joints
Joints:
- joint wheel_left_joint: origin xyz=0 0 0 rpy=0 0 0 -> xyz=-0.075 0.143 0.057215 rpy=0 0 0
- joint wheel_right_joint: origin xyz=0 0 0 rpy=0 0 0 -> xyz=-0.075 -0.143 0.057215 rpy=0 0 0

File: src/r5_2020/urdf/r5_2020.urdf (robot description, URDF)
Before this commit: robot r5_2020, 6 links, 5 joints
Joints:
- joint weapon_joint: origin xyz=0 0 0 rpy=0 0 0 -> xyz=0.183 0 0.0575 rpy=0 0 0
- joint wheel_back_left_joint: origin xyz=0 0 0 rpy=0 0 0 -> xyz=-0.066 -0.1655 0.06 rpy=0 0 0
- joint wheel_back_right_joint: origin xyz=0 0 0 rpy=0 0 0 -> xyz=-0.066 0.1655 0.06 rpy=0 0 0
- joint wheel_front_left_joint: origin xyz=0 0 0 rpy=0 0 0 -> xyz=0.066 0.1655 0.06 rpy=0 0 0
- joint wheel_front_right_joint: origin xyz=0 0 0 rpy=0 0 0 -> xyz=0.066 -0.1655 0.06 rpy=0 0 0

File: src/r6_2020/urdf/r6_2020.urdf (robot description, URDF)
Before this commit: robot r6_2020, 4 links, 3 joints
Links:
- link base_link: mass 10.069 -> 9.337
Joints:
- joint weapon_joint: origin xyz=0 0 0 rpy=0 0 0 -> xyz=0.15788 0.0001548 0.15076 rpy=0 0 0
- joint wheel_left_joint: origin xyz=0 0 0 rpy=0 0 0 -> xyz=0.0185 0.19913 0.07006 rpy=0 0 0
- joint wheel_right_joint: origin xyz=0 0 0 rpy=0 0 0 -> xyz=0.01846 -0.19913 0.07 rpy=0 0 0

File: src/r7_2020/urdf/r7_2020.urdf (robot description, URDF)
Before this commit: robot r7_2020, 3 links, 2 joints
Joints:
- joint wheel_left_joint: origin xyz=0 0 0 rpy=0 0 0 -> xyz=-0.048 0.163 0.0985 rpy=0 0 0
- joint wheel_right_joint: origin xyz=0 0 0 rpy=0 0 0 -> xyz=-0.048 -0.163 0.0985 rpy=0 0 0
